Commit message: correct initialization of mockhardware to urdf

File: armjr_moveit_config/config/arm_jr.ros2_control.xacro (robot description, xacro)
@@ -1,11 +1,20 @@
 <?xml version="1.0"?>
 <robot xmlns:xacro="http://www.ros.org/wiki/xacro">
-    <xacro:macro name="arm_jr_ros2_control" params="name initial_positions_file">
+    <xacro:macro name="arm_jr_ros2_control" params="name initial_positions_file use_mock_hardware">
         <xacro:property name="initial_positions" value="${xacro.load_yaml(initial_positions_file)['initial_positions']}"/>
         <ros2_control name="MockHardwareSystem" type="system">
-            <hardware>
-                <!-- By default, set up controllers for simulation. This won't work on real hardware -->
+            <xacro:unless value="${use_mock_hardware}">
+                <hardware>
+                <plugin>ros2_control_demo_example_2/DiffBotSystemHardware</plugin>
+                <param name="example_param_hw_start_duration_sec">0</param>
+                <param name="example_param_hw_stop_duration_sec">3.0</param>
+                </hardware>
+            </xacro:unless>
+            <xacro:if value="${use_mock_hardware}">
+                <hardware>
                 <plugin>mock_components/GenericSystem</plugin>
-            </hardware>
+                <param name="calculate_dynamics">true</param>
+                </hardware>
+            </xacro:if>
             <joint name="joint1">
                 <command_interface name="position"/>

File: armjr_moveit_config/config/arm_jr.urdf.xacro (robot description, xacro)
@@ -2,8 +2,10 @@
 <robot xmlns:xacro="http://www.ros.org/wiki/xacro" name="arm_jr">
     <xacro:arg name="initial_positions_file" default="initial_positions.yaml" />
+    <xacro:arg name="use_mock_hardware" default="true" />
+    <xacro:arg name="prefix" default="" />
     <!-- Import arm_jr urdf file -->
     <xacro:include filename="$(find cmake_arm_urdf)/urdf/arm_jr.urdf" />
     <!-- Import control_xacro -->
     <xacro:include filename="arm_jr.ros2_control.xacro" />
-    <xacro:arm_jr_ros2_control name="FakeSystem" initial_positions_file="$(arg initial_positions_file)"/>
+    <xacro:arm_jr_ros2_control name="FakeSystem" initial_positions_file="$(arg initial_positions_file)" use_mock_hardware="$(arg use_mock_hardware)"/>
 </robot>

Commit message: correctly launches and ama ble to manally publsih joint trajectory no moveit :(

File: armjr_moveit_config/config/arm_jr.ros2_control.xacro (robot description, xacro)
@@ -6,7 +6,11 @@
             <hardware>
                 <!-- By default, set up controllers for simulation. This won't work on real hardware -->
-                <plugin>mock_components/GenericSystem</plugin>
+                <!-- <plugin>mock_components/GenericSystem</plugin> -->
+                 <plugin>dynamixel_hardware/DynamixelHardware</plugin>
+                    <param name="usb_port">/dev/ttyUSB0</param>
+                    <param name="baud_rate">1000000</param>
             </hardware>
             <joint name="joint1">
+                            <param name="id">1</param>
                 <command_interface name="position"/>
                 <state_interface name="position">
@@ -16,4 +20,5 @@
             </joint>
             <joint name="joint2">
+                                            <param name="id">2</param>
                 <command_interface name="position"/>
                 <state_interface name="position">
@@ -23,4 +28,5 @@
             </joint>
             <joint name="joint3">
+                                            <param name="id">3</param>
                 <command_interface name="position"/>
                 <state_interface name="position">
@@ -30,4 +36,5 @@
             </joint>
             <joint name="joint4">
+                                            <param name="id">4</param>
                 <command_interface name="position"/>
                 <state_interface name="position">
@@ -36,5 +43,6 @@
                 <state_interface name="velocity"/>
             </joint>
-            <joint name="joint5">
+            <!-- <joint name="joint5">
+                <param name="id">5</param>
                 <command_interface name="position"/>
                 <state_interface name="position">
@@ -42,6 +50,7 @@
                 </state_interface>
                 <state_interface name="velocity"/>
-            </joint>
+            </joint> -->
             <joint name="joint6">
+                                            <param name="id">6</param>
                 <command_interface name="position"/>
                 <state_interface name="position">

File: armjr_moveit_config/config/arm_jr.urdf.xacro (robot description, xacro)
@@ -6,4 +6,4 @@
     <!-- Import control_xacro -->
     <xacro:include filename="arm_jr.ros2_control.xacro" />
-    <xacro:arm_jr_ros2_control name="FakeSystem" initial_positions_file="$(arg initial_positions_file)"/>
+    <xacro:arm_jr_ros2_control name="arm_jr_ros2_control" initial_positions_file="$(arg initial_positions_file)"/>
 </robot>

File: cmake_arm_urdf/urdf/arm_jr.urdf (robot description, URDF)
Before this commit: robot arm_jr, 8 links, 7 joints
Joints:
- joint joint5: type revolute -> fixed

Commit message: implement moveit hardware communication

File: armjr_moveit_config/config/arm_jr.ros2_control.xacro (robot description, xacro)
@@ -6,7 +6,11 @@
             <hardware>
                 <!-- By default, set up controllers for simulation. This won't work on real hardware -->
-                <plugin>mock_components/GenericSystem</plugin>
+                <plugin>dynamixel_hardware/DynamixelHardware</plugin>
+  		<param name="usb_port">/dev/ttyUSB0</param>
+  		<param name="baud_rate">1000000</param>
+  		<param name="use_dummy">false</param>
             </hardware>
             <joint name="joint1">
+            	<param name="id">1</param>
                 <command_interface name="position"/>
                 <state_interface name="position">
@@ -16,4 +20,5 @@
             </joint>
             <joint name="joint2">
+            	<param name="id">2</param>
                 <command_interface name="position"/>
                 <state_interface name="position">
@@ -23,4 +28,5 @@
             </joint>
             <joint name="joint3">
+            	<param name="id">3</param>
                 <command_interface name="position"/>
                 <state_interface name="position">
@@ -30,4 +36,5 @@
             </joint>
             <joint name="joint4">
+            	<param name="id">4</param>
                 <command_interface name="position"/>
                 <state_interface name="position">
@@ -36,5 +43,7 @@
                 <state_interface name="velocity"/>
             </joint>
+            <!--
             <joint name="joint5">
+            	<param name="id">5</param>
                 <command_interface name="position"/>
                 <state_interface name="position">
@@ -43,5 +52,7 @@
                 <state_interface name="velocity"/>
             </joint>
+            -->
             <joint name="joint6">
+            	<param name="id">6</param>
                 <command_interface name="position"/>
                 <state_interface name="position">

File: cmake_arm_urdf/urdf/low_cost_robot.urdf (robot description, URDF)
Before this commit: robot low-cost-arm, 6 links, 5 joints
Links:
- removed link elbow-to-wrist-motor-reference_v1_1
- removed link gripper-moving-part-dumb_v2_1
- removed link gripper-static-motor_v2_1
- removed link shoulder-to-elbow-motor_v1_1
- added link elbow_to_wrist_reference, mass 0.02059907441055582; collision mesh filename=package://dof_arm/meshes/elbow_to_wrist_extension.stl scale=0.001 0.001 0.001; visual mesh filename=package://dof_arm/meshes/elbow_to_wrist_extension.stl scale=0.001 0.001 0.001
- added link gripper_moving_part, mass 0.013583445641331692; collision mesh filename=package://dof_arm/meshes/gripper_moving_part.stl scale=0.001 0.001 0.001; visual mesh filename=package://dof_arm/meshes/gripper_moving_part.stl scale=0.001 0.001 0.001
- added link gripper_static_part, mass 0.030801959916802346; collision mesh filename=package://dof_arm/meshes/gripper_static_part.stl scale=0.001 0.001 0.001; visual mesh filename=package://dof_arm/meshes/gripper_static_part.stl scale=0.001 0.001 0.001
- added link shoulder_to_elbow, mass 0.05261369068977079; collision mesh filename=package://dof_arm/meshes/shouler_to_elbow.stl scale=0.001 0.001 0.001; visual mesh filename=package://dof_arm/meshes/shouler_to_elbow.stl scale=0.001 0.001 0.001
- link base_link: geometry collision mesh filename=package://dof_arm/meshes/base.stl scale=0.001 0.001 0.001; visual mesh filename=package://dof_arm/meshes/base.stl scale=0.001 0.001 0.001
- link first-bracket-motor_1: geometry collision mesh filename=package://dof_arm/meshes/shoulder_rotation.stl scale=0.001 0.001 0.001; visual mesh filename=package://dof_arm/meshes/shoulder_rotation.stl scale=0.001 0.001 0.001
Joints:
- added joint Revolute 4: type continuous, parent shoulder_to_elbow, child elbow_to_wrist_reference, origin xyz=0.03375 0.0 0.05 rpy=0 0 0, axis 1.0 0.0 0.0, limit effort=5.0 velocity=1.5
- joint Revolute 3: child shoulder-to-elbow-motor_v1_1 -> shoulder_to_elbow
- joint Revolute 5: child elbow-to-wrist-motor-reference_v1_1 -> gripper_static_part; parent shoulder-to-elbow-motor_v1_1 -> elbow_to_wrist_reference
- joint Revolute 6: child gripper-static-motor_v2_1 -> gripper_moving_part; parent elbow-to-wrist-motor-reference_v1_1 -> gripper_static_part
- joint Revolute 7: child gripper-moving-part-dumb_v2_1 -> gripper_moving_part; parent gripper-static-motor_v2_1 -> gripper_static_part

Commit message: add fix for motor 5

File: armjr_moveit_config/config/arm_jr.ros2_control.xacro (robot description, xacro)
@@ -43,5 +43,4 @@
                 <state_interface name="velocity"/>
             </joint>
-            <!--
             <joint name="joint5">
             	<param name="id">5</param>
@@ -52,5 +51,4 @@
                 <state_interface name="velocity"/>
             </joint>
-            -->
             <joint name="joint6">
             	<param name="id">6</param>

File: cmake_arm_urdf/urdf/arm_jr.urdf (robot description, URDF)
Before this commit: robot arm_jr, 8 links, 7 joints
Joints:
- joint joint5: axis 0 -1 0 -> 0 1 0; type fixed -> revolute
- joint joint6: axis 0 0 -1 -> 0 0 1
